File: Bluetooth.sch (KiCad schematic (older format))
At the start: 18 parts, among them J4 Conn_01x03, U12 SW_AKIDUKI

Commit message: 改版中
Parts:
- removed C20: 100u/6.3V, Capacitor_THT:CP_Radial_D5.0mm_P2.00mm, symbol Device:CP_Small
- removed C21, C22, C23, C24: 22u/16V, Capacitor_THT:CP_Radial_D5.0mm_P2.00mm, symbol Device:CP_Small
- added C36: 220u/6.3V, Capacitor_SMD:C_1210_3225Metric_Pad1.42x2.65mm_HandSolder, symbol Device:C_Small
- added C39, C47, C53, C54: 22u/25V, Capacitor_SMD:C_0805_2012Metric_Pad1.15x1.40mm_HandSolder, symbol Device:C_Small
Connections:
- net labels added: BM62_MFB, BM62_SYS_PWR, mix_out_L, mix_out_R
- net labels removed: BM64_MFB, BM64_SYS_PWR, BT_Line_out_L, BT_Line_out_R
Changed lines of the file:
@@
 Wire Wire Line
 	6550 3700 7000 3700
-$Comp
-L Device:CP_Small C22
-U 1 1 5EECB5D4
-P 4750 3800
-F 0 "C22" V 4850 3550 50  0000 C CNN
-F 1 "22u/16V" V 4850 3850 50  0000 C CNN
-F 2 "Capacitor_THT:CP_Radial_D5.0mm_P2.00mm" H 4750 3800 50  0001 C CNN
-F 3 "~" H 4750 3800 50  0001 C CNN
-	1    4750 3800
-	0    1    1    0
-$EndComp
-$Comp
-L Device:CP_Small C21
-U 1 1 5EECC49D
-P 4750 3600
-F 0 "C21" V 4650 3350 50  0000 C CNN
-F 1 "22u/16V" V 4650 3650 50  0000 C CNN
-F 2 "Capacitor_THT:CP_Radial_D5.0mm_P2.00mm" H 4750 3600 50  0001 C CNN
-F 3 "~" H 4750 3600 50  0001 C CNN
-	1    4750 3600
-	0    1    1    0
-$EndComp
 Wire Wire Line
 	4850 3800 5050 3800
@@
 Wire Wire Line
 	6800 3200 6550 3200
-$Comp
-L Device:CP_Small C20
-U 1 1 5EEDF73E
-P 4500 5050
-F 0 "C20" H 4600 4950 50  0000 C CNN
-F 1 "100u/6.3V" H 4500 4850 50  0000 C CNN
-F 2 "Capacitor_THT:CP_Radial_D5.0mm_P2.00mm" H 4500 5050 50  0001 C CNN
-F 3 "~" H 4500 5050 50  0001 C CNN
-	1    4500 5050
-	1    0    0    -1
-$EndComp
 Wire Wire Line
 	4500 4950 4500 4900
@@
 Wire Wire Line
 	4800 5200 4800 5250
-$Comp
-L Device:CP_Small C24
-U 1 1 5EEE4A13
-P 4750 4450
-F 0 "C24" V 4850 4200 50  0000 C CNN
-F 1 "22u/16V" V 4850 4500 50  0000 C CNN
-F 2 "Capacitor_THT:CP_Radial_D5.0mm_P2.00mm" H 4750 4450 50  0001 C CNN
-F 3 "~" H 4750 4450 50  0001 C CNN
-	1    4750 4450
-	0    1    1    0
-$EndComp
-$Comp
-L Device:CP_Small C23
-U 1 1 5EEE4C91
-P 4750 4250
-F 0 "C23" V 4650 4000 50  0000 C CNN
-F 1 "22u/16V" V 4650 4300 50  0000 C CNN
-F 2 "Capacitor_THT:CP_Radial_D5.0mm_P2.00mm" H 4750 4250 50  0001 C CNN
-F 3 "~" H 4750 4250 50  0001 C CNN
-	1    4750 4250
-	0    1    1    0
-$EndComp
 Wire Wire Line
 	4850 4250 4950 4250
@@
 $EndComp
 Text GLabel 2850 4450 0    50   Input ~ 0
-BT_Line_out_L
+mix_out_L
 Text GLabel 2850 4250 0    50   Input ~ 0
-BT_Line_out_R
+mix_out_R
 Wire Wire Line
 	3350 4450 4650 4450
@@
 $EndComp
 Text GLabel 6750 3500 2    50   Input ~ 0
-BM64_MFB
+BM62_MFB
 Wire Wire Line
 	6750 3500 6550 3500
 Text GLabel 6750 3300 2    50   Input ~ 0
-BM64_SYS_PWR
+BM62_SYS_PWR
 Wire Wire Line
 	6750 3300 6550 3300
 Text GLabel 7400 3600 2    50   Input ~ 0
-BM64_SYS_PWR
+BM62_SYS_PWR
 Wire Wire Line
 	7400 3600 7350 3600
@@
 	7350 3600 7050 3600
 Text GLabel 10000 3300 2    50   Input ~ 0
-BM64_MFB
+BM62_MFB
 $Comp
 L power:GND #PWR?
@@
 $EndComp
 Text GLabel 9000 3300 0    50   Input ~ 0
-BM64_SYS_PWR
+BM62_SYS_PWR
 Wire Wire Line
 	9050 3200 9050 3300
@@
 Wire Wire Line
 	9950 3600 9950 3650
+$Comp
+L Device:C_Small C?
+U 1 1 5F52E8E7
+P 4500 5050
+AR Path="/5F52E8E7" Ref="C?"  Part="1"
+AR Path="/5EF8073C/5F52E8E7" Ref="C?"  Part="1"
+AR Path="/5F64C24C/5F52E8E7" Ref="C36"  Part="1"
+F 0 "C36" H 4300 4950 50  0000 L CNN
+F 1 "220u/6.3V" H 4250 4800 50  0000 L CNN
+F 2 "Capacitor_SMD:C_1210_3225Metric_Pad1.42x2.65mm_HandSolder" H 4500 5050 50  0001 C CNN
+F 3 "~" H 4500 5050 50  0001 C CNN
+	1    4500 5050
+	1    0    0    -1
+$EndComp
+$Comp
+L Device:C_Small C?
+U 1 1 5F5315A0
+P 4750 4450
+AR Path="/5F5315A0" Ref="C?"  Part="1"
+AR Path="/5EF8073C/5F5315A0" Ref="C?"  Part="1"
+AR Path="/5F64C24C/5F5315A0" Ref="C54"  Part="1"
+F 0 "C54" V 4800 4250 50  0000 L CNN
+F 1 "22u/25V" V 4900 4150 50  0000 L CNN
+F 2 "Capacitor_SMD:C_0805_2012Metric_Pad1.15x1.40mm_HandSolder" H 4750 4450 50  0001 C CNN
+F 3 "~" H 4750 4450 50  0001 C CNN
+	1    4750 4450
+	0    1    1    0
+$EndComp
+$Comp
+L Device:C_Small C?
+U 1 1 5F532B95
+P 4750 4250
+AR Path="/5F532B95" Ref="C?"  Part="1"
+AR Path="/5EF8073C/5F532B95" Ref="C?"  Part="1"
+AR Path="/5F64C24C/5F532B95" Ref="C53"  Part="1"
+F 0 "C53" V 4550 4050 50  0000 L CNN
+F 1 "22u/25V" V 4650 3950 50  0000 L CNN
+F 2 "Capacitor_SMD:C_0805_2012Metric_Pad1.15x1.40mm_HandSolder" H 4750 4250 50  0001 C CNN
+F 3 "~" H 4750 4250 50  0001 C CNN
+	1    4750 4250
+	0    1    1    0
+$EndComp
+$Comp
+L Device:C_Small C?
+U 1 1 5F532E51
+P 4750 3800
+AR Path="/5F532E51" Ref="C?"  Part="1"
+AR Path="/5EF8073C/5F532E51" Ref="C?"  Part="1"
+AR Path="/5F64C24C/5F532E51" Ref="C47"  Part="1"
+F 0 "C47" V 4800 3600 50  0000 L CNN
+F 1 "22u/25V" V 4900 3500 50  0000 L CNN
+F 2 "Capacitor_SMD:C_0805_2012Metric_Pad1.15x1.40mm_HandSolder" H 4750 3800 50  0001 C CNN
+F 3 "~" H 4750 3800 50  0001 C CNN
+	1    4750 3800
+	0    1    1    0
+$EndComp
+$Comp
+L Device:C_Small C?
+U 1 1 5F53311B
+P 4750 3600
+AR Path="/5F53311B" Ref="C?"  Part="1"
+AR Path="/5EF8073C/5F53311B" Ref="C?"  Part="1"
+AR Path="/5F64C24C/5F53311B" Ref="C39"  Part="1"
+F 0 "C39" V 4550 3400 50  0000 L CNN
+F 1 "22u/25V" V 4650 3300 50  0000 L CNN
+F 2 "Capacitor_SMD:C_0805_2012Metric_Pad1.15x1.40mm_HandSolder" H 4750 3600 50  0001 C CNN
+F 3 "~" H 4750 3600 50  0001 C CNN
+	1    4750 3600
+	0    1    1    0
+$EndComp
 $EndSCHEMATC

Commit message: Rev.A 作成中
Parts:
- removed C25: 0.1u, Capacitor_SMD:C_0603_1608Metric_Pad1.05x0.95mm_HandSolder, symbol Device:C_Small
- renumbered C36 to C27, C39 to C28, C47 to C29, C53 to C30, C54 to C31, D4 to D2, D5 to D3, D2 to D4, D3 to D5, J4 to J5, R22 to R21, U12 to U8
Other:
- moved on the sheet: C27
Changed lines of the file:
@@
 P 4800 4850
 AR Path="/5EE15687/5EEA5FCE" Ref="#PWR?"  Part="1"
-AR Path="/5F64C24C/5EEA5FCE" Ref="#PWR038"  Part="1"
-F 0 "#PWR038" H 4800 4700 50  0001 C CNN
+AR Path="/5F64C24C/5EEA5FCE" Ref="#PWR043"  Part="1"
+F 0 "#PWR043" H 4800 4700 50  0001 C CNN
 F 1 "+5VD" H 4650 4900 50  0000 C CNN
 F 2 "" H 4800 4850 50  0001 C CNN
@@
 	1    0    0    -1
 $EndComp
-$Comp
-L Device:C_Small C?
-U 1 1 5EEA9878
-P 4800 5050
-AR Path="/5EEA9878" Ref="C?"  Part="1"
-AR Path="/5EF8073C/5EEA9878" Ref="C?"  Part="1"
-AR Path="/5F64C24C/5EEA9878" Ref="C25"  Part="1"
-F 0 "C25" H 4900 5100 50  0000 L CNN
-F 1 "0.1u" H 4900 5000 50  0000 L CNN
-F 2 "Capacitor_SMD:C_0603_1608Metric_Pad1.05x0.95mm_HandSolder" H 4800 5050 50  0001 C CNN
-F 3 "~" H 4800 5050 50  0001 C CNN
-	1    4800 5050
-	1    0    0    -1
-$EndComp
 Wire Wire Line
 	5050 4900 4800 4900
@@
 AR Path="/5EE15687/5EEABA35" Ref="#PWR?"  Part="1"
 AR Path="/5EEABA35" Ref="#PWR?"  Part="1"
-AR Path="/5F64C24C/5EEABA35" Ref="#PWR039"  Part="1"
-F 0 "#PWR039" H 4800 5000 50  0001 C CNN
+AR Path="/5F64C24C/5EEABA35" Ref="#PWR044"  Part="1"
+F 0 "#PWR044" H 4800 5000 50  0001 C CNN
 F 1 "GND" H 4805 5077 50  0000 C CNN
 F 2 "" H 4800 5250 50  0001 C CNN
@@
 	-1   0    0    -1
 $EndComp
-Wire Wire Line
-	4800 5150 4800 5200
 $Comp
 L power:GND #PWR?
@@
 AR Path="/5EE15687/5EEAC597" Ref="#PWR?"  Part="1"
 AR Path="/5EEAC597" Ref="#PWR?"  Part="1"
-AR Path="/5F64C24C/5EEAC597" Ref="#PWR040"  Part="1"
-F 0 "#PWR040" H 6850 4450 50  0001 C CNN
+AR Path="/5F64C24C/5EEAC597" Ref="#PWR045"  Part="1"
+F 0 "#PWR045" H 6850 4450 50  0001 C CNN
 F 1 "GND" H 6855 4527 50  0000 C CNN
 F 2 "" H 6850 4700 50  0001 C CNN
@@
 	4550 3800 4650 3800
 $Comp
-L Connector_Generic:Conn_01x03 J4
+L Connector_Generic:Conn_01x03 J5
 U 1 1 5EED3116
 P 7150 4200
-F 0 "J4" H 7230 4242 50  0000 L CNN
+F 0 "J5" H 7230 4242 50  0000 L CNN
 F 1 "Conn_01x03" H 7230 4151 50  0000 L CNN
 F 2 "Connector_PinHeader_2.54mm:PinHeader_1x03_P2.54mm_Vertical" H 7150 4200 50  0001 C CNN
@@
 AR Path="/5EE15687/5EEDB113" Ref="#PWR?"  Part="1"
 AR Path="/5EEDB113" Ref="#PWR?"  Part="1"
-AR Path="/5F64C24C/5EEDB113" Ref="#PWR041"  Part="1"
-F 0 "#PWR041" H 7050 2800 50  0001 C CNN
+AR Path="/5F64C24C/5EEDB113" Ref="#PWR046"  Part="1"
+F 0 "#PWR046" H 7050 2800 50  0001 C CNN
 F 1 "GND" H 7050 2900 50  0000 C CNN
 F 2 "" H 7050 3050 50  0001 C CNN
@@
 Wire Wire Line
 	6800 3200 6550 3200
-Wire Wire Line
-	4500 4950 4500 4900
-Wire Wire Line
-	4500 4900 4800 4900
-Wire Wire Line
-	4800 5200 4500 5200
-Wire Wire Line
-	4500 5200 4500 5150
-Connection ~ 4800 5200
-Wire Wire Line
-	4800 5200 4800 5250
 Wire Wire Line
 	4850 4250 4950 4250
@@
 AR Path="/5EE15687/5EF20964" Ref="#PWR?"  Part="1"
 AR Path="/5EF20964" Ref="#PWR?"  Part="1"
-AR Path="/5F64C24C/5EF20964" Ref="#PWR036"  Part="1"
-F 0 "#PWR036" H 3350 4950 50  0001 C CNN
+AR Path="/5F64C24C/5EF20964" Ref="#PWR042"  Part="1"
+F 0 "#PWR042" H 3350 4950 50  0001 C CNN
 F 1 "GND" H 3355 5027 50  0000 C CNN
 F 2 "" H 3350 5200 50  0001 C CNN
@@
 Uart
 $Comp
-L toripoyo:SW_AKIDUKI U12
+L toripoyo:SW_AKIDUKI U8
 U 1 1 5EFC8780
 P 9700 3350
-F 0 "U12" H 9900 3450 50  0000 C CNN
+F 0 "U8" H 9900 3450 50  0000 C CNN
 F 1 "SW_AKIDUKI" H 9900 3550 50  0000 C CNN
 F 2 "hastech:SW_AKZK" H 9600 3450 50  0001 C CNN
@@
 	3350 4450 4650 4450
 $Comp
-L Device:D_Zener D2
+L Device:D_Zener D4
 U 1 1 5F32D539
 P 3350 4650
-F 0 "D2" V 3304 4730 50  0000 L CNN
+F 0 "D4" V 3304 4730 50  0000 L CNN
 F 1 "VESD01-02V-G-08" V 3395 4730 50  0000 L CNN
 F 2 "Diode_SMD:D_SOD-523" H 3350 4650 50  0001 C CNN
@@
 $EndComp
 $Comp
-L Device:D_Zener D3
+L Device:D_Zener D5
 U 1 1 5F3345A1
 P 3350 5000
-F 0 "D3" V 3396 4920 50  0000 R CNN
+F 0 "D5" V 3396 4920 50  0000 R CNN
 F 1 "VESD01-02V-G-08" V 3305 4920 50  0000 R CNN
 F 2 "Diode_SMD:D_SOD-523" H 3350 5000 50  0001 C CNN
@@
 	3350 5150 3350 5200
 $Comp
-L Device:D_Zener D4
+L Device:D_Zener D2
 U 1 1 5F34202B
 P 3350 3700
-F 0 "D4" V 3304 3780 50  0000 L CNN
+F 0 "D2" V 3304 3780 50  0000 L CNN
 F 1 "VESD01-02V-G-08" V 3395 3780 50  0000 L CNN
 F 2 "Diode_SMD:D_SOD-523" H 3350 3700 50  0001 C CNN
@@
 $EndComp
 $Comp
-L Device:D_Zener D5
+L Device:D_Zener D3
 U 1 1 5F342035
 P 3350 4050
-F 0 "D5" V 3396 3970 50  0000 R CNN
+F 0 "D3" V 3396 3970 50  0000 R CNN
 F 1 "VESD01-02V-G-08" V 3305 3970 50  0000 R CNN
 F 2 "Diode_SMD:D_SOD-523" H 3350 4050 50  0001 C CNN
@@
 AR Path="/5EE15687/5F1934C6" Ref="#PWR?"  Part="1"
 AR Path="/5F1934C6" Ref="#PWR?"  Part="1"
-AR Path="/5F64C24C/5F1934C6" Ref="#PWR046"  Part="1"
-F 0 "#PWR046" H 3150 3350 50  0001 C CNN
+AR Path="/5F64C24C/5F1934C6" Ref="#PWR041"  Part="1"
+F 0 "#PWR041" H 3150 3350 50  0001 C CNN
 F 1 "GND" H 3155 3427 50  0000 C CNN
 F 2 "" H 3150 3600 50  0001 C CNN
@@
 	3150 3600 3150 3500
 $Comp
-L Device:R_Small R22
+L Device:R_Small R21
 U 1 1 5F19625D
 P 9950 3500
-F 0 "R22" H 9800 3550 50  0000 C CNN
+F 0 "R21" H 9800 3550 50  0000 C CNN
 F 1 "2k" H 9800 3450 50  0000 C CNN
 F 2 "Resistor_SMD:R_0603_1608Metric_Pad1.05x0.95mm_HandSolder" H 9950 3500 50  0001 C CNN
@@
 AR Path="/5EE15687/5F1B7F37" Ref="#PWR?"  Part="1"
 AR Path="/5F1B7F37" Ref="#PWR?"  Part="1"
-AR Path="/5F64C24C/5F1B7F37" Ref="#PWR050"  Part="1"
-F 0 "#PWR050" H 9950 3400 50  0001 C CNN
+AR Path="/5F64C24C/5F1B7F37" Ref="#PWR047"  Part="1"
+F 0 "#PWR047" H 9950 3400 50  0001 C CNN
 F 1 "GND" H 9950 3500 50  0000 C CNN
 F 2 "" H 9950 3650 50  0001 C CNN
@@
 L Device:C_Small C?
 U 1 1 5F52E8E7
-P 4500 5050
+P 4800 5050
 AR Path="/5F52E8E7" Ref="C?"  Part="1"
 AR Path="/5EF8073C/5F52E8E7" Ref="C?"  Part="1"
-AR Path="/5F64C24C/5F52E8E7" Ref="C36"  Part="1"
-F 0 "C36" H 4300 4950 50  0000 L CNN
-F 1 "220u/6.3V" H 4250 4800 50  0000 L CNN
-F 2 "Capacitor_SMD:C_1210_3225Metric_Pad1.42x2.65mm_HandSolder" H 4500 5050 50  0001 C CNN
-F 3 "~" H 4500 5050 50  0001 C CNN
-	1    4500 5050
+AR Path="/5F64C24C/5F52E8E7" Ref="C27"  Part="1"
+F 0 "C27" H 4950 5050 50  0000 L CNN
+F 1 "220u/6.3V" H 4850 4950 50  0000 L CNN
+F 2 "Capacitor_SMD:C_1210_3225Metric_Pad1.42x2.65mm_HandSolder" H 4800 5050 50  0001 C CNN
+F 3 "~" H 4800 5050 50  0001 C CNN
+	1    4800 5050
 	1    0    0    -1
 $EndComp
@@
 AR Path="/5F5315A0" Ref="C?"  Part="1"
 AR Path="/5EF8073C/5F5315A0" Ref="C?"  Part="1"
-AR Path="/5F64C24C/5F5315A0" Ref="C54"  Part="1"
-F 0 "C54" V 4800 4250 50  0000 L CNN
+AR Path="/5F64C24C/5F5315A0" Ref="C31"  Part="1"
+F 0 "C31" V 4800 4250 50  0000 L CNN
 F 1 "22u/25V" V 4900 4150 50  0000 L CNN
 F 2 "Capacitor_SMD:C_0805_2012Metric_Pad1.15x1.40mm_HandSolder" H 4750 4450 50  0001 C CNN
@@
 AR Path="/5F532B95" Ref="C?"  Part="1"
 AR Path="/5EF8073C/5F532B95" Ref="C?"  Part="1"
-AR Path="/5F64C24C/5F532B95" Ref="C53"  Part="1"
-F 0 "C53" V 4550 4050 50  0000 L CNN
+AR Path="/5F64C24C/5F532B95" Ref="C30"  Part="1"
+F 0 "C30" V 4550 4050 50  0000 L CNN
 F 1 "22u/25V" V 4650 3950 50  0000 L CNN
 F 2 "Capacitor_SMD:C_0805_2012Metric_Pad1.15x1.40mm_HandSolder" H 4750 4250 50  0001 C CNN
@@
 AR Path="/5F532E51" Ref="C?"  Part="1"
 AR Path="/5EF8073C/5F532E51" Ref="C?"  Part="1"
-AR Path="/5F64C24C/5F532E51" Ref="C47"  Part="1"
-F 0 "C47" V 4800 3600 50  0000 L CNN
+AR Path="/5F64C24C/5F532E51" Ref="C29"  Part="1"
+F 0 "C29" V 4800 3600 50  0000 L CNN
 F 1 "22u/25V" V 4900 3500 50  0000 L CNN
 F 2 "Capacitor_SMD:C_0805_2012Metric_Pad1.15x1.40mm_HandSolder" H 4750 3800 50  0001 C CNN
@@
 AR Path="/5F53311B" Ref="C?"  Part="1"
 AR Path="/5EF8073C/5F53311B" Ref="C?"  Part="1"
-AR Path="/5F64C24C/5F53311B" Ref="C39"  Part="1"
-F 0 "C39" V 4550 3400 50  0000 L CNN
+AR Path="/5F64C24C/5F53311B" Ref="C28"  Part="1"
+F 0 "C28" V 4550 3400 50  0000 L CNN
 F 1 "22u/25V" V 4650 3300 50  0000 L CNN
 F 2 "Capacitor_SMD:C_0805_2012Metric_Pad1.15x1.40mm_HandSolder" H 4750 3600 50  0001 C CNN
@@
 	0    1    1    0
 $EndComp
+Wire Wire Line
+	4800 5150 4800 5250
 $EndSCHEMATC

Commit message: Rev.A 完成
Parts:
- removed C30, C31: 22u/25V, Capacitor_SMD:C_0805_2012Metric_Pad1.15x1.40mm_HandSolder, symbol Device:C_Small
- removed D2, D3, D4, D5: VESD01-02V-G-08, Diode_SMD:D_SOD-523, symbol Device:D_Zener
- removed R19, R20: 2k, Resistor_SMD:R_0603_1608Metric_Pad1.05x0.95mm_HandSolder, symbol Device:R_Small
- removed U8: SW_AKIDUKI, hastech:SW_AKZK, symbol toripoyo:SW_AKIDUKI
- added SW6: SW_Push, Button_Switch_THT:SW_PUSH_6mm, symbol Switch:SW_Push
Connections:
- net GND is gone; now on net GNDD: ANT1.23 (GND_1), ANT1.37 (GND_2), C27.2, J5.3 (Pin_3), R21.1
- net BM62_MFB: now also SW6.2
- net BM62_SYS_PWR: now also SW6.1
- net BT_Mic_Out_P: now reaches ANT1.11 (MIC1_P)
- net BT_Mic_Out_N: now reaches ANT1.12 (MIC1_N)
- net GNDD: now reaches ANT1.3 (P3_0)
- no-connect marks 27 -> 26
Other:
- note removed: "Input Protection"

Commit message: Rev.B 改版完了
Parts:
- removed J5: Conn_01x03, Connector_PinHeader_2.54mm:PinHeader_1x03_P2.54mm_Vertical, symbol Connector_Generic:Conn_01x03
- added TP1, TP2, TP3, TP4, TP5, TP6, TP7: TestPoint, TestPoint:TestPoint_Pad_D1.0mm, symbol Connector:TestPoint
Connections:
- net GNDD: now also TP3.1; no longer ANT1.3 (P3_0)
- net VDDIO: now reaches ANT1.19 (VDD_IO)
- net VDDIO: now also TP7.1
- net EAN: now reaches ANT1.2 (EAN)
- net EAN: now also TP6.1
- net P2_4: now reaches ANT1.29 (P2_4)
- net P2_4: now also TP4.1
- net at ANT1.32 (HCI_TXD): now also TP1.1
- net at ANT1.33 (HCI_RXD): now also TP2.1
- net P2_0: now reaches ANT1.4 (P2_0)
- new net P0_2: TP5.1
- no-connect marks 26 -> 23
Other:
- note added: "Update"
- note removed: "Uart"
- moved on the sheet: C27
Changed lines of the file:
@@
 L power:+5VD #PWR?
 U 1 1 5EEA5FCE
-P 4800 4850
+P 4525 4850
 AR Path="/5EE15687/5EEA5FCE" Ref="#PWR?"  Part="1"
 AR Path="/5F64C24C/5EEA5FCE" Ref="#PWR043"  Part="1"
-F 0 "#PWR043" H 4800 4700 50  0001 C CNN
-F 1 "+5VD" H 4650 4900 50  0000 C CNN
-F 2 "" H 4800 4850 50  0001 C CNN
-F 3 "" H 4800 4850 50  0001 C CNN
-	1    4800 4850
-	1    0    0    -1
-$EndComp
-Wire Wire Line
-	5050 4900 4800 4900
-Wire Wire Line
-	4800 4850 4800 4900
-Wire Wire Line
-	4800 4900 4800 4950
-Connection ~ 4800 4900
+F 0 "#PWR043" H 4525 4700 50  0001 C CNN
+F 1 "+5VD" H 4375 4900 50  0000 C CNN
+F 2 "" H 4525 4850 50  0001 C CNN
+F 3 "" H 4525 4850 50  0001 C CNN
+	1    4525 4850
+	1    0    0    -1
+$EndComp
+Wire Wire Line
+	5050 4900 4525 4900
+Wire Wire Line
+	4525 4850 4525 4900
+Wire Wire Line
+	4525 4900 4525 4950
+Connection ~ 4525 4900
 $Comp
 L Device:LED D6
@@
 Wire Wire Line
 	4550 3800 4650 3800
-$Comp
-L Connector_Generic:Conn_01x03 J5
-U 1 1 5EED3116
-P 7150 4200
-F 0 "J5" H 7230 4242 50  0000 L CNN
-F 1 "Conn_01x03" H 7230 4151 50  0000 L CNN
-F 2 "Connector_PinHeader_2.54mm:PinHeader_1x03_P2.54mm_Vertical" H 7150 4200 50  0001 C CNN
-F 3 "~" H 7150 4200 50  0001 C CNN
-	1    7150 4200
-	1    0    0    -1
-$EndComp
-Wire Wire Line
-	6850 4700 6850 4600
-Wire Wire Line
-	6850 4600 6550 4600
-Wire Wire Line
-	6850 4600 6850 4300
-Wire Wire Line
-	6850 4300 6950 4300
-Connection ~ 6850 4600
-Wire Wire Line
-	6950 4200 6550 4200
-Wire Wire Line
-	6550 4100 6950 4100
+Wire Wire Line
+	6750 4700 6750 4600
+Wire Wire Line
+	6750 4600 6550 4600
+Wire Wire Line
+	6550 4100 6800 4100
 Wire Wire Line
 	7050 3050 7050 3000
@@
 	6800 3200 6550 3200
 NoConn ~ 5050 3000
-NoConn ~ 5050 3100
-NoConn ~ 5050 3300
 NoConn ~ 5050 3400
 NoConn ~ 5050 3500
@@
 NoConn ~ 5050 4600
 NoConn ~ 5050 4700
-NoConn ~ 5050 4800
 NoConn ~ 6550 4700
 NoConn ~ 6550 4800
@@
 NoConn ~ 6550 4300
 NoConn ~ 6550 4000
-NoConn ~ 6550 3900
-NoConn ~ 6550 3800
 NoConn ~ 6550 3400
 NoConn ~ 6550 3100
 NoConn ~ 6550 3000
-Text Notes 7100 4450 0    50   ~ 0
-Uart
+Text Notes 7000 4550 0    50   ~ 0
+Update
 $Comp
 L Device:R_Small R21
@@
 L Device:C_Small C?
 U 1 1 5F52E8E7
-P 4800 5050
+P 4525 5050
 AR Path="/5F52E8E7" Ref="C?"  Part="1"
 AR Path="/5EF8073C/5F52E8E7" Ref="C?"  Part="1"
 AR Path="/5F64C24C/5F52E8E7" Ref="C27"  Part="1"
-F 0 "C27" H 4950 5050 50  0000 L CNN
-F 1 "220u/6.3V" H 4850 4950 50  0000 L CNN
-F 2 "Capacitor_SMD:C_1210_3225Metric_Pad1.42x2.65mm_HandSolder" H 4800 5050 50  0001 C CNN
-F 3 "~" H 4800 5050 50  0001 C CNN
-	1    4800 5050
+F 0 "C27" H 4675 5050 50  0000 L CNN
+F 1 "220u/6.3V" H 4575 4950 50  0000 L CNN
+F 2 "Capacitor_SMD:C_1210_3225Metric_Pad1.42x2.65mm_HandSolder" H 4525 5050 50  0001 C CNN
+F 3 "~" H 4525 5050 50  0001 C CNN
+	1    4525 5050
 	1    0    0    -1
 $EndComp
@@
 $EndComp
 Wire Wire Line
-	4800 5150 4800 5250
-Wire Wire Line
-	4650 3100 4650 3050
-Wire Wire Line
-	4650 3050 4850 3050
-Wire Wire Line
-	4850 3050 4850 3200
-Wire Wire Line
-	4850 3200 5050 3200
+	4525 5150 4525 5250
 Text GLabel 4550 4000 0    50   Input ~ 0
 BT_Mic_Out_P
@@
 L power:GNDD #PWR047
 U 1 1 60010975
-P 6850 4700
-F 0 "#PWR047" H 6850 4450 50  0001 C CNN
-F 1 "GNDD" H 6854 4545 50  0000 C CNN
-F 2 "" H 6850 4700 50  0001 C CNN
-F 3 "" H 6850 4700 50  0001 C CNN
-	1    6850 4700
+P 6750 4700
+F 0 "#PWR047" H 6750 4450 50  0001 C CNN
+F 1 "GNDD" H 6754 4545 50  0000 C CNN
+F 2 "" H 6750 4700 50  0001 C CNN
+F 3 "" H 6750 4700 50  0001 C CNN
+	1    6750 4700
 	1    0    0    -1
 $EndComp
@@
 $EndComp
 $Comp
-L power:GNDD #PWR045
-U 1 1 60013883
-P 4650 3100
-F 0 "#PWR045" H 4650 2850 50  0001 C CNN
-F 1 "GNDD" H 4654 2945 50  0000 C CNN
-F 2 "" H 4650 3100 50  0001 C CNN
-F 3 "" H 4650 3100 50  0001 C CNN
-	1    4650 3100
-	1    0    0    -1
-$EndComp
-$Comp
 L power:GNDD #PWR046
 U 1 1 60014E3A
-P 4800 5250
-F 0 "#PWR046" H 4800 5000 50  0001 C CNN
-F 1 "GNDD" H 4804 5095 50  0000 C CNN
-F 2 "" H 4800 5250 50  0001 C CNN
-F 3 "" H 4800 5250 50  0001 C CNN
-	1    4800 5250
+P 4525 5250
+F 0 "#PWR046" H 4525 5000 50  0001 C CNN
+F 1 "GNDD" H 4529 5095 50  0000 C CNN
+F 2 "" H 4525 5250 50  0001 C CNN
+F 3 "" H 4525 5250 50  0001 C CNN
+	1    4525 5250
 	1    0    0    -1
 $EndComp
@@
 Wire Wire Line
 	9250 3300 9425 3300
+NoConn ~ 5050 3200
+Text GLabel 4925 3100 0    50   Input ~ 0
+EAN
+Wire Wire Line
+	4925 3100 5050 3100
+Text GLabel 7550 4300 2    50   Input ~ 0
+EAN
+Wire Wire Line
+	7550 4300 7450 4300
+Text GLabel 6600 3800 2    50   Input ~ 0
+P2_4
+Text GLabel 4925 3300 0    50   Input ~ 0
+P2_0
+Wire Wire Line
+	5050 3300 4925 3300
+Text GLabel 7550 4200 2    50   Input ~ 0
+P0_2
+Wire Wire Line
+	6600 3800 6550 3800
+NoConn ~ 6550 3900
+Text GLabel 7550 4100 2    50   Input ~ 0
+P2_4
+Wire Wire Line
+	7550 4100 7450 4100
+Wire Wire Line
+	7550 4200 7450 4200
+Text GLabel 4950 4800 0    50   Input ~ 0
+VDDIO
+Wire Wire Line
+	4950 4800 5050 4800
+Text GLabel 7550 4400 2    50   Input ~ 0
+VDDIO
+Wire Wire Line
+	7550 4400 7450 4400
+$Comp
+L Connector:TestPoint TP1
+U 1 1 5FD801E4
+P 6800 4100
+F 0 "TP1" V 6800 4288 50  0000 L CNN
+F 1 "TestPoint" V 6845 4288 50  0001 L CNN
+F 2 "TestPoint:TestPoint_Pad_D1.0mm" H 7000 4100 50  0001 C CNN
+F 3 "~" H 7000 4100 50  0001 C CNN
+	1    6800 4100
+	0    1    1    0
+$EndComp
+Wire Wire Line
+	6800 4200 6550 4200
+$Comp
+L Connector:TestPoint TP2
+U 1 1 5FD8971F
+P 6800 4200
+F 0 "TP2" V 6800 4388 50  0000 L CNN
+F 1 "TestPoint" V 6845 4388 50  0001 L CNN
+F 2 "TestPoint:TestPoint_Pad_D1.0mm" H 7000 4200 50  0001 C CNN
+F 3 "~" H 7000 4200 50  0001 C CNN
+	1    6800 4200
+	0    1    1    0
+$EndComp
+$Comp
+L Connector:TestPoint TP3
+U 1 1 5FD89D67
+P 6800 4300
+F 0 "TP3" V 6800 4488 50  0000 L CNN
+F 1 "TestPoint" V 6845 4488 50  0001 L CNN
+F 2 "TestPoint:TestPoint_Pad_D1.0mm" H 7000 4300 50  0001 C CNN
+F 3 "~" H 7000 4300 50  0001 C CNN
+	1    6800 4300
+	0    1    1    0
+$EndComp
+Wire Wire Line
+	6750 4600 6750 4300
+Wire Wire Line
+	6750 4300 6800 4300
+Connection ~ 6750 4600
+$Comp
+L Connector:TestPoint TP4
+U 1 1 5FD94007
+P 7450 4100
+F 0 "TP4" V 7450 4350 50  0000 C CNN
+F 1 "TestPoint" V 7495 4288 50  0001 L CNN
+F 2 "TestPoint:TestPoint_Pad_D1.0mm" H 7650 4100 50  0001 C CNN
+F 3 "~" H 7650 4100 50  0001 C CNN
+	1    7450 4100
+	0    -1   -1   0
+$EndComp
+$Comp
+L Connector:TestPoint TP5
+U 1 1 5FD9737C
+P 7450 4200
+F 0 "TP5" V 7450 4450 50  0000 C CNN
+F 1 "TestPoint" V 7495 4388 50  0001 L CNN
+F 2 "TestPoint:TestPoint_Pad_D1.0mm" H 7650 4200 50  0001 C CNN
+F 3 "~" H 7650 4200 50  0001 C CNN
+	1    7450 4200
+	0    -1   -1   0
+$EndComp
+$Comp
+L Connector:TestPoint TP6
+U 1 1 5FD97613
+P 7450 4300
+F 0 "TP6" V 7450 4550 50  0000 C CNN
+F 1 "TestPoint" V 7495 4488 50  0001 L CNN
+F 2 "TestPoint:TestPoint_Pad_D1.0mm" H 7650 4300 50  0001 C CNN
+F 3 "~" H 7650 4300 50  0001 C CNN
+	1    7450 4300
+	0    -1   -1   0
+$EndComp
+$Comp
+L Connector:TestPoint TP7
+U 1 1 5FD977CD
+P 7450 4400
+F 0 "TP7" V 7450 4650 50  0000 C CNN
+F 1 "TestPoint" V 7495 4588 50  0001 L CNN
+F 2 "TestPoint:TestPoint_Pad_D1.0mm" H 7650 4400 50  0001 C CNN
+F 3 "~" H 7650 4400 50  0001 C CNN
+	1    7450 4400
+	0    -1   -1   0
+$EndComp
 $EndSCHEMATC
