File: Input.sch (KiCad schematic (older format))
At the start: 37 parts, among them J10 Conn_01x03, J5 AudioJack3, J6 Conn_01x03, J7 AudioJack3, J8 Conn_01x03, J9 AudioJack3, SW2 SW_DPDT_x2, SW3 SW_DPDT_x2, U11 NJM4580CG

Commit message: 改版中
Parts:
- removed C36, C39: 22u/16V, Capacitor_THT:CP_Radial_D5.0mm_P2.00mm, symbol Device:CP_Small
- removed C40, C41: 0.47u, Capacitor_THT:C_Rect_L11.0mm_W4.2mm_P10.00mm_MKT, symbol Device:CP_Small
- removed J10, J6, J8: Conn_01x03, Connector_PinHeader_2.54mm:PinHeader_1x03_P2.54mm_Vertical, symbol Connector_Generic:Conn_01x03
- added C40, C41: 1u, Capacitor_SMD:C_0603_1608Metric_Pad1.05x0.95mm_HandSolder, symbol Device:C_Small
- added C55, C56: 22u/25V, Capacitor_SMD:C_0805_2012Metric_Pad1.15x1.40mm_HandSolder, symbol Device:C_Small
- C50, C51: value option footprint -> 1u
- J5, J7, J9: value AudioJack3 -> PJ-3420
- R41, R42: value 100k -> 10k
- RV3, RV4, RV5: value RV10kA -> RK0972-A10K
- SW2, SW3: value SW_DPDT_x2 -> OS202011MA0QN1
Connections:
- wire segments 160 -> 131
Other:
- moved on the sheet: C50, C51, RV5

Commit message: Rev.A 作成中
Parts:
- removed C44: 0.1u, Capacitor_SMD:C_0603_1608Metric_Pad1.05x0.95mm_HandSolder, symbol Device:C_Small
- renumbered C55 to C39, C37 to C40, C38 to C41, C56 to C42, C50 to C43, C51 to C44, C42 to C47, C43 to C48, C40 to C49, C41 to C50, J7 to J6, J5 to J7, J9 to J8, R37 to R27, R38 to R28, R39 to R29, R40 to R30, R41 to R31, R42 to R32, R43 to R33, R44 to R34, R46 to R35, R45 to R36, R47 to R37, R48 to R38, RV3 to RV2, RV4 to RV3, RV5 to RV4
Other:
- moved on the sheet: U11C

Commit message: Rev.A 完成
Parts:
- added C26, C30: 1u, Capacitor_SMD:C_0603_1608Metric_Pad1.05x0.95mm_HandSolder, symbol Device:C_Small
- added R48, R49: 10k, Resistor_SMD:R_0603_1608Metric_Pad1.05x0.95mm_HandSolder, symbol Device:R_Small
- added R50, R51: 1k, Resistor_SMD:R_0603_1608Metric_Pad1.05x0.95mm_HandSolder, symbol Device:R_Small
- added R52, R53: 100, Resistor_SMD:R_0603_1608Metric_Pad1.05x0.95mm_HandSolder, symbol Device:R_Small
- added SW4, SW5: OS202011MA0QN1, digikey-download:OS202011MA0QN1, symbol Switch:SW_DPDT_x2
- R27, R30: value 4.7 -> 470
Connections:
- net GND: now also C26.1, R50.2, R51.2, SW5.3 (C), SW5.6 (C)
- net at C43.1, R31.1, U11.3 (+): now also SW5.5 (B)
- net at C43.2, J8.T, R28.2: now also SW4.6 (C)
- net at C44.2, J8.R, R29.2: now also SW4.3 (C)
- net at C44.1, R32.1, U11.5 (+): now also SW5.2 (B)
- new net: R52.1, SW4.2 (B)
- new net: C30.2, R52.2, R53.2
- new net: R53.1, SW4.5 (B)
- new net: R49.1, R51.1, SW4.1 (A)
- new net: R48.1, R50.1, SW4.4 (A)
- new net BT_Mic_Out_N: C26.2
- new net BT_Mic_Out_P: C30.1
- new net mix_out_L: R49.2
- new net mix_out_R: R48.2
- no-connect marks 2 -> 4
Other:
- note added: "Mic Mute"
- note added: "Send Select\nMix/Mic Only"
- moved on the sheet: C39, C40, C41, C42, C43, C44, C45, C46, C47, C48, C49, C50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

Commit message: Rev.B 改版完了
Parts:
- R48, R49: value 10k -> 100k
Connections:
- net BT_Mic_Out_P: now also SW5.2 (B), SW5.5 (B)
- net at C43.1, R31.1, U11.3 (+): no longer SW5.5 (B)
- net at C44.1, R32.1, U11.5 (+): no longer SW5.2 (B)
Other:
- note added: "Mic Send Mute"
- note removed: "Mic Mute"
- moved on the sheet: SW5A, SW5B
Changed lines of the file:
@@
 	0    1    1    0
 $EndComp
-Wire Wire Line
-	6625 2300 6775 2300
 $Comp
 L Device:C_Small C?
@@
 	0    1    1    0
 $EndComp
-Wire Wire Line
-	6625 1300 7200 1300
 Wire Wire Line
 	6225 1300 6425 1300
@@
 AR Path="/5EF8073C/5FBE4065" Ref="C26"  Part="1"
 F 0 "C26" V 4900 2475 50  0000 L CNN
-F 1 "1u" V 4825 2475 50  0000 L CNN
+F 1 "1u" V 4825 2500 50  0000 L CNN
 F 2 "Capacitor_SMD:C_0603_1608Metric_Pad1.05x0.95mm_HandSolder" H 5025 2600 50  0001 C CNN
 F 3 "~" H 5025 2600 50  0001 C CNN
@@
 AR Path="/5EF8073C/5FC075DE" Ref="R49"  Part="1"
 F 0 "R49" V 5025 3300 50  0000 L CNN
-F 1 "10k" V 5025 3475 50  0000 L CNN
+F 1 "100k" V 5025 3475 50  0000 L CNN
 F 2 "Resistor_SMD:R_0603_1608Metric_Pad1.05x0.95mm_HandSolder" H 4925 3500 50  0001 C CNN
 F 3 "~" H 4925 3500 50  0001 C CNN
@@
 AR Path="/5EF8073C/5FC07D0A" Ref="R48"  Part="1"
 F 0 "R48" V 4825 3175 50  0000 L CNN
-F 1 "10k" V 4825 3350 50  0000 L CNN
+F 1 "100k" V 4825 3350 50  0000 L CNN
 F 2 "Resistor_SMD:R_0603_1608Metric_Pad1.05x0.95mm_HandSolder" H 4925 3375 50  0001 C CNN
 F 3 "~" H 4925 3375 50  0001 C CNN
@@
 Wire Wire Line
 	4825 3500 4725 3500
-Text Notes 6925 3800 0    50   ~ 0
-Mic Mute
+Text Notes 5775 5625 0    50   ~ 0
+Mic Send Mute
 Wire Notes Line
 	3775 3950 575  3950
@@
 L Switch:SW_DPDT_x2 SW5
 U 1 1 5FF34C52
-P 6775 3250
-F 0 "SW5" V 6750 3075 50  0000 C CNN
-F 1 "OS202011MA0QN1" V 7175 3625 50  0000 C CNN
-F 2 "digikey-download:OS202011MA0QN1" H 6775 3250 50  0001 C CNN
-F 3 "https://www.digikey.jp/product-detail/ja/c-k/OS202011MA0QN1/CKN9563-ND/1981434" H 6775 3250 50  0001 C CNN
-	1    6775 3250
+P 5700 5075
+F 0 "SW5" V 5675 4900 50  0000 C CNN
+F 1 "OS202011MA0QN1" V 6100 5450 50  0000 C CNN
+F 2 "digikey-download:OS202011MA0QN1" H 5700 5075 50  0001 C CNN
+F 3 "https://www.digikey.jp/product-detail/ja/c-k/OS202011MA0QN1/CKN9563-ND/1981434" H 5700 5075 50  0001 C CNN
+	1    5700 5075
 	0    1    1    0
 $EndComp
@@
 L Switch:SW_DPDT_x2 SW5
 U 2 1 5FF34C5C
-P 7200 3250
-F 0 "SW5" V 7175 3075 50  0000 C CNN
-F 1 "OS202011MA0QN1" V 7350 2725 50  0001 C CNN
-F 2 "digikey-download:OS202011MA0QN1" H 7200 3250 50  0001 C CNN
-F 3 "https://www.digikey.jp/product-detail/ja/c-k/OS202011MA0QN1/CKN9563-ND/1981434" H 7200 3250 50  0001 C CNN
-	2    7200 3250
-	0    1    1    0
-$EndComp
-Wire Wire Line
-	6775 3050 6775 2300
-Connection ~ 6775 2300
-Wire Wire Line
-	6775 2300 7700 2300
-Wire Wire Line
-	7200 3050 7200 1300
-Connection ~ 7200 1300
-Wire Wire Line
-	7200 1300 7700 1300
-NoConn ~ 6875 3450
-NoConn ~ 7300 3450
+P 6125 5075
+F 0 "SW5" V 6100 4900 50  0000 C CNN
+F 1 "OS202011MA0QN1" V 6275 4550 50  0001 C CNN
+F 2 "digikey-download:OS202011MA0QN1" H 6125 5075 50  0001 C CNN
+F 3 "https://www.digikey.jp/product-detail/ja/c-k/OS202011MA0QN1/CKN9563-ND/1981434" H 6125 5075 50  0001 C CNN
+	2    6125 5075
+	0    1    1    0
+$EndComp
+NoConn ~ 5800 5275
+NoConn ~ 6225 5275
 $Comp
 L power:GND #PWR?
 U 1 1 5FF842E9
-P 6675 3600
+P 5600 5425
 AR Path="/5EE15687/5FF842E9" Ref="#PWR?"  Part="1"
 AR Path="/5FF842E9" Ref="#PWR?"  Part="1"
 AR Path="/5EF8073C/5FF842E9" Ref="#PWR095"  Part="1"
-F 0 "#PWR095" H 6675 3350 50  0001 C CNN
-F 1 "GND" H 6680 3427 50  0000 C CNN
-F 2 "" H 6675 3600 50  0001 C CNN
-F 3 "" H 6675 3600 50  0001 C CNN
-	1    6675 3600
+F 0 "#PWR095" H 5600 5175 50  0001 C CNN
+F 1 "GND" H 5605 5252 50  0000 C CNN
+F 2 "" H 5600 5425 50  0001 C CNN
+F 3 "" H 5600 5425 50  0001 C CNN
+	1    5600 5425
 	-1   0    0    -1
 $EndComp
 Wire Wire Line
-	6675 3600 6675 3525
-Wire Wire Line
-	6675 3525 7100 3525
-Wire Wire Line
-	7100 3525 7100 3450
-Connection ~ 6675 3525
-Wire Wire Line
-	6675 3525 6675 3450
+	5600 5425 5600 5350
+Wire Wire Line
+	5600 5350 6025 5350
+Wire Wire Line
+	6025 5350 6025 5275
+Connection ~ 5600 5350
+Wire Wire Line
+	5600 5350 5600 5275
+Wire Wire Line
+	6625 2300 7700 2300
+Wire Wire Line
+	6625 1300 7700 1300
+Wire Wire Line
+	5700 4875 5700 4750
+Connection ~ 5700 4750
+Wire Wire Line
+	5700 4750 6125 4750
+Wire Wire Line
+	6125 4750 6125 4875
 $EndSCHEMATC
