File: LevelMeter.sch (KiCad schematic (older format))
At the start: 28 parts, among them U10 NJM4580CG, U8 NJM4580CG, U9 NJM4580CG

Commit message: 改版中
Parts:
- removed C32, C33, C34: 0.1u, Capacitor_SMD:C_0603_1608Metric_Pad1.05x0.95mm_HandSolder, symbol Device:C_Small
- removed C35, C47: 0.47u, Capacitor_THT:CP_Radial_D5.0mm_P2.00mm, symbol Device:CP_Small
- removed C48, C49: option_footprint, Capacitor_SMD:C_0603_1608Metric_Pad1.05x0.95mm_HandSolder, symbol Device:C_Small
- removed D10, D12: SS2040, Diode_SMD:D_SOD-123, symbol Device:D
- removed D11, D13: LED_RED, LED_SMD:LED_0603_1608Metric_Pad1.05x0.95mm_HandSolder, symbol Device:LED
- removed R24: 470k, Resistor_SMD:R_0603_1608Metric_Pad1.05x0.95mm_HandSolder, symbol Device:R_Small
- removed R36: 470, Resistor_SMD:R_0603_1608Metric_Pad1.05x0.95mm_HandSolder, symbol Device:R_Small
- removed unit 3 of U10
- removed unit 2 of U9
- removed unit 1 of U9
- added D10: LED_ORANGE, LED_SMD:LED_0603_1608Metric_Pad1.05x0.95mm_HandSolder, symbol Device:LED
- added D13, D14: 1N4148, Diode_SMD:D_SOD-123, symbol Device:D
- added R23: 1.2k, Resistor_SMD:R_0603_1608Metric_Pad1.05x0.95mm_HandSolder, symbol Device:R_Small
- D8, D9: value SS2040 -> 1N4148
- R21: value 470k -> 22k
- R31: value 4.7k -> 22k
- R32: value 4.7k -> 1.2k
- R35: value 470 -> 1k
- renumbered U10 to U9
Connections:
- wire segments 125 -> 71
Other:
- note added: "-10dBV"
- note removed: "220ms"
- note removed: "Peak\n1/2 Vcc"
- moved on the sheet: C26, C27, C28, C29, C30, C31, R31, R32, R35, U8C, U9A, U9B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

Commit message: Rev.A 作成中
Parts:
- removed C26, C27, C28, C29, C30, C31: 0.1u, Capacitor_SMD:C_0603_1608Metric_Pad1.05x0.95mm_HandSolder, symbol Device:C_Small
- removed D13, D14, D8, D9: 1N4148, Diode_SMD:D_SOD-123, symbol Device:D
- removed R21: 22k, Resistor_SMD:R_0603_1608Metric_Pad1.05x0.95mm_HandSolder, symbol Device:R_Small
- removed R23: 1.2k, Resistor_SMD:R_0603_1608Metric_Pad1.05x0.95mm_HandSolder, symbol Device:R_Small
- removed U8, U9: NJM4580CG, Package_SO:SOP-8_3.9x4.9mm_P1.27mm, symbol Amplifier_Operational:NJM4558
- added C33, C34: 0.1u, Capacitor_SMD:C_0603_1608Metric_Pad1.05x0.95mm_HandSolder, symbol Device:C_Small
- added J10, J9: Conn_01x03, Connector_PinSocket_2.54mm:PinSocket_1x03_P2.54mm_Vertical, symbol Connector_Generic:Conn_01x03
- added R24, R39: 33k, Resistor_SMD:R_0603_1608Metric_Pad1.05x0.95mm_HandSolder, symbol Device:R_Small
- added R25, R40: 8.2k, Resistor_SMD:R_0603_1608Metric_Pad1.05x0.95mm_HandSolder, symbol Device:R_Small
- added R41: 22k, Resistor_SMD:R_0603_1608Metric_Pad1.05x0.95mm_HandSolder, symbol Device:R_Small
- added R42: 1.2k, Resistor_SMD:R_0603_1608Metric_Pad1.05x0.95mm_HandSolder, symbol Device:R_Small
- added U9: LM339PWR, Package_SO:TSSOP-14_4.4x5mm_P0.65mm, symbol toripoyo:LM339PWR
- R26: renamed from R35; value 1k -> 4.7k
- renumbered D10 to D12, R31 to R22, R32 to R23
Connections:
- net +9VA: now also R26.1, C33.1, R24.2, U9.3 (Vcc)
- net -9VA: now also C34.1, R40.1, R42.1, U9.12 (GND)
- net GND: now also C33.2, C34.2, R25.1, R39.2, R41.2; no longer D12.1 (K)
- net mix_out_L: now also U9.5 (In2+), U9.6 (In1-)
- net mix_out_R: now also U9.11 (In4+), U9.8 (In3-)
- net at R22.1, R23.2: now also J9.3 (Pin_3)
- new net: J9.1 (Pin_1), R24.1, R25.2
- new net: J10.3 (Pin_3), R41.1, R42.2
- new net: J10.1 (Pin_1), R39.1, R40.2
- new net: D12.1 (K), U9.1 (Out1), U9.13 (Out4), U9.14 (Out3), U9.2 (Out2)
- new net vref_out_+: J9.2 (Pin_2), U9.7 (In1+), U9.9 (In3+)
- new net vref_out_-: J10.2 (Pin_2), U9.10 (In4-), U9.4 (In2-)
Other:
- moved on the sheet: D12, R22, R23, R26

Commit message: Rev.A 完成
Parts:
- removed J10, J9: Conn_01x03, Connector_PinSocket_2.54mm:PinSocket_1x03_P2.54mm_Vertical, symbol Connector_Generic:Conn_01x03
- added C13, C14: 47u, Capacitor_SMD:C_1210_3225Metric_Pad1.42x2.65mm_HandSolder, symbol Device:C_Small
- added C23, C24, C25, C3, C6, C9: 0.1u, Capacitor_SMD:C_0603_1608Metric_Pad1.05x0.95mm_HandSolder, symbol Device:C_Small
- added D2, D4: LED_GREEN, LED_SMD:LED_0603_1608Metric_Pad1.05x0.95mm_HandSolder, symbol Device:LED
- added D3: LED_RED, LED_SMD:LED_0603_1608Metric_Pad1.05x0.95mm_HandSolder, symbol Device:LED
- added JP2: UserShort, Jumper:SolderJumper-2_P1.3mm_Open_RoundedPad1.0x1.5mm, symbol kamiya:UserShort
- added R19: 33k, Resistor_SMD:R_0603_1608Metric_Pad1.05x0.95mm_HandSolder, symbol Device:R_Small
- added R20: 1.2k, Resistor_SMD:R_0603_1608Metric_Pad1.05x0.95mm_HandSolder, symbol Device:R_Small
- added R43, R44, R45: 4.7k, Resistor_SMD:R_0603_1608Metric_Pad1.05x0.95mm_HandSolder, symbol Device:R_Small
- added R46, R47: 100, Resistor_SMD:R_0603_1608Metric_Pad1.05x0.95mm_HandSolder, symbol Device:R_Small
- added U10: LM339PWR, Package_SO:TSSOP-14_4.4x5mm_P0.65mm, symbol toripoyo:LM339PWR
- D12: value LED_ORANGE -> LED_RED
- R24: value 33k -> 1.2k
- R25: value 8.2k -> 33k
- R39: value 33k -> 100
- R40: value 8.2k -> 100
Connections:
- net vref_out_+ is gone; now on net vref_out_+_-10dBv: U9.7 (In1+), U9.9 (In3+)
- net +9VA: now also R39.2, R40.2, C13.1, R19.2, R43.1, R44.1, R45.1; no longer C33.1, R24.2, U9.3 (Vcc)
- net -9VA: now also R25.1, R41.1, C14.2, R46.2, R47.2; no longer C34.1, R40.1, R42.1, U9.12 (GND)
- net GND: now also JP2.1; no longer C33.2, C34.2, R23.1, R25.1, R39.2, R41.2
- net mix_out_L: now also U10.5 (In2+), U10.6 (In1-)
- net mix_out_R: now also U10.11 (In4+), U10.8 (In3-)
- net vref_out_+_-10dBv: now reaches R22.1, R23.2
- net vref_out_+_-10dBv: now also C3.1
- net vref_out_-_-13dBv: now reaches R24.1, R25.2
- net vref_out_-_-13dBv: now also C23.1, U10.10 (In4-), U10.4 (In2-)
- net GND2: now reaches R42.2
- net GND2: now also C33.2, C34.2, R23.1, R24.2, C13.2, C14.1, C23.2, C24.2, C25.2, C3.2, C6.2, C9.2, JP2.2, R20.1; no longer R41.1
- net at R39.1: now also C33.1, U9.3 (Vcc); no longer R40.2
- net at D12.1 (K), U9.1 (Out1), U9.2 (Out2): no longer U9.13 (Out4), U9.14 (Out3)
- net vref_out_- renamed vref_out_-_-10dBv
- net vref_out_-_-10dBv: now also R41.2, R42.1, C9.1
- new net: C34.1, R46.1, U9.12 (GND)
- new net: D3.1 (K), U9.13 (Out4), U9.14 (Out3)
- new net: D3.2 (A), R44.2
- new net: D2.2 (A), R43.2
- new net: D2.1 (K), U10.1 (Out1), U10.2 (Out2)
- new net: C24.1, R40.1, U10.3 (Vcc)
- new net: C25.1, R47.1, U10.12 (GND)
- new net: D4.1 (K), U10.13 (Out4), U10.14 (Out3)
- new net: D4.2 (A), R45.2
- new net vref_out_+_-13dBv: C6.1, R19.1, R20.2, U10.7 (In1+), U10.9 (In3+)
Other:
- note added: "-10dBv"
- note added: "-13dBv"
- note removed: "-10dBV"
- moved on the sheet: C33, C34, D12, R22, R23, R26, R41, R42, U9

Commit message: Rev.B 改版完了
Parts:
- R26, R44: value 4.7k -> 10k
- R43, R45: value 4.7k -> 33k
Other:
- note added: "adjust by own"
Changed lines of the file:
@@
 P 6450 1625
 F 0 "R26" H 6600 1675 50  0000 C CNN
-F 1 "4.7k" H 6600 1575 50  0000 C CNN
+F 1 "10k" H 6600 1575 50  0000 C CNN
 F 2 "Resistor_SMD:R_0603_1608Metric_Pad1.05x0.95mm_HandSolder" H 6450 1625 50  0001 C CNN
 F 3 "~" H 6450 1625 50  0001 C CNN
@@
 P 7600 1625
 F 0 "R44" H 7450 1675 50  0000 C CNN
-F 1 "4.7k" H 7450 1575 50  0000 C CNN
+F 1 "10k" H 7450 1575 50  0000 C CNN
 F 2 "Resistor_SMD:R_0603_1608Metric_Pad1.05x0.95mm_HandSolder" H 7600 1625 50  0001 C CNN
 F 3 "~" H 7600 1625 50  0001 C CNN
@@
 P 6450 4200
 F 0 "R43" H 6600 4250 50  0000 C CNN
-F 1 "4.7k" H 6600 4150 50  0000 C CNN
+F 1 "33k" H 6600 4150 50  0000 C CNN
 F 2 "Resistor_SMD:R_0603_1608Metric_Pad1.05x0.95mm_HandSolder" H 6450 4200 50  0001 C CNN
 F 3 "~" H 6450 4200 50  0001 C CNN
@@
 P 7600 4200
 F 0 "R45" H 7450 4250 50  0000 C CNN
-F 1 "4.7k" H 7450 4150 50  0000 C CNN
+F 1 "33k" H 7450 4150 50  0000 C CNN
 F 2 "Resistor_SMD:R_0603_1608Metric_Pad1.05x0.95mm_HandSolder" H 7600 4200 50  0001 C CNN
 F 3 "~" H 7600 4200 50  0001 C CNN
@@
 Wire Wire Line
 	3025 5275 3025 5175
+Text Notes 6525 4075 0    50   ~ 0
+adjust by own
+Text Notes 6525 1500 0    50   ~ 0
+adjust by own
 $EndSCHEMATC
