File: Mixer.kicad_pcb (KiCad board)
At the start: 2 copper layers, 135 x 59 mm, 139 parts, among them J1 PJ-3420, J2 PJ-3420, J3 Conn_02x02_Counter_Clockwise, J4 USB_B_Micro, J5 Conn_01x03, J6 PJ-3420, J7 PJ-3420, J8 PJ-3420, SW1 2MS1-T1-B2-M7-S-E, SW2 OS202011MA0QN1, SW3 OS202011MA0QN1, SW4 OS202011MA0QN1, SW5 OS202011MA0QN1, SW6 SW_Push, U1 NJM4580CG, U10 LM339PWR, U11 NJM4580CG, U2 NJM4580CG, U3 NJM4580CG, U4 MCW03, U5 MCW03, U6 NJM7809, U7 NJM7909, U9 LM339PWR

Commit message: Rev.B 改版完了
Parts:
- removed J3: Conn_02x02_Counter_Clockwise, Connector_PinHeader_2.54mm:PinHeader_2x02_P2.54mm_Vertical
- removed J5: Conn_01x03, Connector_PinHeader_2.54mm:PinHeader_1x03_P2.54mm_Vertical
- removed JP1: UserShort, Jumper:SolderJumper-2_P1.3mm_Open_RoundedPad1.0x1.5mm
- added C19: 22p, Capacitor_SMD:C_0603_1608Metric_Pad1.05x0.95mm_HandSolder, B.Cu at (175.0, 94.8)
- added C20: 22p, Capacitor_SMD:C_0603_1608Metric_Pad1.05x0.95mm_HandSolder, B.Cu at (188.3, 95.1)
- added SW7: SW_SPDT, Button_Switch_THT:SW_Slide_1P2T_CK_OS102011MS2Q, F.Cu at (126.0, 98.8)
- added TP1: TestPoint, TestPoint:TestPoint_Pad_D1.0mm, B.Cu at (129.5, 79.4)
- added TP2: TestPoint, TestPoint:TestPoint_Pad_D1.0mm, B.Cu at (127.1, 79.4)
- added TP3: TestPoint, TestPoint:TestPoint_Pad_D1.0mm, B.Cu at (129.5, 83.6)
- added TP4: TestPoint, TestPoint:TestPoint_Pad_D1.0mm, B.Cu at (129.5, 81.4)
- added TP6: TestPoint, TestPoint:TestPoint_Pad_D1.0mm, B.Cu at (121.8, 73.0)
- added TP7: TestPoint, TestPoint:TestPoint_Pad_D1.0mm, B.Cu at (127.1, 83.6)
- C31: value 0.1u -> 22u/25V; footprint Capacitor_SMD:C_0603_1608Metric_Pad1.05x0.95mm_HandSolder -> Capacitor_SMD:C_0805_2012Metric_Pad1.15x1.40mm_HandSolder
- R26, R44: value 4.7k -> 10k
- R43, R45: value 4.7k -> 33k
- R48, R49: value 10k -> 100k
- R54: value 100 -> 1k
- moved R8 0.20 mm to (188.3, 95.1)
Connections:
- ANT1 pad 19: (no net) -> VDDIO
- ANT1 pad 2: (no net) -> EAN
- ANT1 pad 29: (no net) -> P2_4
- ANT1 pad 3: GNDD -> (no net)
- SW5 pad 2: Net-(C44-Pad1) -> BT_Mic_Out_P
- SW5 pad 5: Net-(C43-Pad1) -> BT_Mic_Out_P
Routing:
- net BT_Mic_Out_P: track 151.7 -> 182.5 mm
- net Net-(C44-Pad1): track 34.6 -> 15.2 mm, vias 3 -> 2
- net Net-(C43-Pad1): track 45.1 -> 28.8 mm
- net Net-(ANT1-Pad32): track 19.2 -> 4.31 mm
- net Net-(ANT1-Pad33): track 21.1 -> 7.24 mm
- net VDDIO: track 0.00 -> 5.77 mm, vias 0 -> 1
- net P2_4: track 0.00 -> 3.66 mm, vias 0 -> 1
- net EAN: track 0.00 -> 3.15 mm, vias 0 -> 1
- net Net-(C19-Pad1): track 6.77 -> 9.59 mm, vias 0 -> 1
- net Net-(C20-Pad1): track 6.89 -> 9.17 mm, vias 0 -> 1
- net Net-(C19-Pad2): track 11.1 -> 12.4 mm, vias 0 -> 1
- net Net-(C49-Pad1): track 41.5 -> 40.5 mm
- net Net-(C20-Pad2): track 11.0 -> 11.9 mm, vias 0 -> 1
- net BM62_SYS_PWR: track 48.7 -> 49.3 mm
- net GNDD: vias 41 -> 40
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Other:
- board text added: "2020/12/19 Rev.B toripoyo"
- board text added: "EAN"
- board text added: "GND Isolate"
- board text added: "GNDD"
- board text added: "OFF ON"
- board text added: "P2_4"
- board text added: "Rx"
- board text added: "Tx"
- board text added: "VDDIO"
- board text removed: "-Isolate |Common"
- board text removed: "2020/11/24 Rev.A poyo"
- board text removed: "GND Rx Tx"
