File: Mixer.sch (KiCad schematic (older format))
At the start: 36 parts, among them J1 AudioJack3, J2 AudioJack3, U1 NJM4580CG, U2 NJM4580CG, U3 NJM4580CG

Commit message: 改版中
Parts:
- removed RV2: RV10kA, toripoyo:RD925G-QA1, symbol Device:R_POT_Dual_Separate
- J1, J2: value AudioJack3 -> PJ-3420
- R13, R14: value 10k -> 33k
- RV1: value RV10kA -> RK0972-A10K
Connections:
- net BT_Line_out_L is gone; now on net mix_out_L: R15.2
- net BT_Line_out_R is gone; now on net mix_out_R: R16.2
Other:
- note removed: "Bluetooth/Line Out"
Changed lines of the file:
@@
 Sheet 1 5
 Title "Anarogu Mikisa-"
-Date "2020-06-11"
-Rev ""
+Date "2020-08-18"
+Rev "B"
 Comp "Poyo"
 Comment1 ""
@@
 P 5850 2050
 F 0 "R13" V 6046 2050 50  0000 C CNN
-F 1 "10k" V 5955 2050 50  0000 C CNN
+F 1 "33k" V 5955 2050 50  0000 C CNN
 F 2 "Resistor_SMD:R_0603_1608Metric_Pad1.05x0.95mm_HandSolder" H 5850 2050 50  0001 C CNN
 F 3 "~" H 5850 2050 50  0001 C CNN
@@
 P 5850 3850
 F 0 "R14" V 6046 3850 50  0000 C CNN
-F 1 "10k" V 5955 3850 50  0000 C CNN
+F 1 "33k" V 5955 3850 50  0000 C CNN
 F 2 "Resistor_SMD:R_0603_1608Metric_Pad1.05x0.95mm_HandSolder" H 5850 3850 50  0001 C CNN
 F 3 "~" H 5850 3850 50  0001 C CNN
@@
 P 8250 2400
 F 0 "RV1" H 8181 2446 50  0000 R CNN
-F 1 "RV10kA" H 8181 2355 50  0000 R CNN
+F 1 "RK0972-A10K" H 8181 2355 50  0000 R CNN
 F 2 "toripoyo:RD925G-QA1" H 8250 2400 50  0001 C CNN
 F 3 "~" H 8250 2400 50  0001 C CNN
@@
 P 8250 1500
 F 0 "RV1" H 8181 1546 50  0000 R CNN
-F 1 "RV10kA" H 8181 1455 50  0000 R CNN
+F 1 "RK0972-A10K" H 8181 1455 50  0000 R CNN
 F 2 "toripoyo:RD925G-QA1" H 8250 1500 50  0001 C CNN
 F 3 "~" H 8250 1500 50  0001 C CNN
@@
 Wire Wire Line
 	9400 2250 9400 2350
-$Comp
-L Device:R_POT_Dual_Separate RV2
-U 1 1 5EF9C197
-P 9900 5700
-F 0 "RV2" H 9831 5746 50  0000 R CNN
-F 1 "RV10kA" H 9831 5655 50  0000 R CNN
-F 2 "toripoyo:RD925G-QA1" H 9900 5700 50  0001 C CNN
-F 3 "~" H 9900 5700 50  0001 C CNN
-	1    9900 5700
-	1    0    0    1
-$EndComp
-Text GLabel 8250 5450 0    50   Input ~ 0
-mix_out_L
-Wire Wire Line
-	8250 5450 8350 5450
-Wire Wire Line
-	8350 5450 8350 5550
-$Comp
-L power:GND #PWR?
-U 1 1 5EF9C1B1
-P 8350 6000
-AR Path="/5EE15687/5EF9C1B1" Ref="#PWR?"  Part="1"
-AR Path="/5EF9C1B1" Ref="#PWR016"  Part="1"
-F 0 "#PWR016" H 8350 5750 50  0001 C CNN
-F 1 "GND" H 8355 5827 50  0000 C CNN
-F 2 "" H 8350 6000 50  0001 C CNN
-F 3 "" H 8350 6000 50  0001 C CNN
-	1    8350 6000
-	-1   0    0    -1
-$EndComp
-Wire Wire Line
-	8350 6000 8350 5850
-$Comp
-L Device:R_POT_Dual_Separate RV2
-U 2 1 5EF9C1C6
-P 8350 5700
-F 0 "RV2" H 8281 5746 50  0000 R CNN
-F 1 "RV10kA" H 8281 5655 50  0000 R CNN
-F 2 "toripoyo:RD925G-QA1" H 8350 5700 50  0001 C CNN
-F 3 "~" H 8350 5700 50  0001 C CNN
-	2    8350 5700
-	1    0    0    1
-$EndComp
-Text GLabel 9800 5450 0    50   Input ~ 0
-mix_out_R
-Wire Wire Line
-	9800 5450 9900 5450
-Wire Wire Line
-	9900 5450 9900 5550
-$Comp
-L power:GND #PWR?
-U 1 1 5EF9C1DF
-P 9900 6000
-AR Path="/5EE15687/5EF9C1DF" Ref="#PWR?"  Part="1"
-AR Path="/5EF9C1DF" Ref="#PWR019"  Part="1"
-F 0 "#PWR019" H 9900 5750 50  0001 C CNN
-F 1 "GND" H 9905 5827 50  0000 C CNN
-F 2 "" H 9900 6000 50  0001 C CNN
-F 3 "" H 9900 6000 50  0001 C CNN
-	1    9900 6000
-	-1   0    0    -1
-$EndComp
-Wire Wire Line
-	9900 6000 9900 5850
-Text GLabel 8700 5700 2    50   Input ~ 0
-BT_Line_out_L
-Text GLabel 10250 5700 2    50   Input ~ 0
-BT_Line_out_R
 $Sheet
 S 1150 2200 800  300
@@
 $EndSheet
 Wire Wire Line
-	10050 5700 10250 5700
-Wire Wire Line
-	8500 5700 8700 5700
-Wire Wire Line
 	8400 1900 9200 1900
 Wire Wire Line
@@
 Text Notes 9600 3900 0    79   ~ 0
 Line Out
-Text Notes 8250 5250 0    79   ~ 0
-Bluetooth/Line Out
 $Comp
 L Device:C_Small C1
@@
 P 10000 2150
 F 0 "J2" H 9720 2083 50  0000 R CNN
-F 1 "AudioJack3" H 9720 2174 50  0000 R CNN
+F 1 "PJ-3420" H 9720 2174 50  0000 R CNN
 F 2 "toripoyo:PJ-3420" H 10000 2150 50  0001 C CNN
 F 3 "~" H 10000 2150 50  0001 C CNN
@@
 P 9250 4050
 F 0 "J1" H 8970 3983 50  0000 R CNN
-F 1 "AudioJack3" H 8970 4074 50  0000 R CNN
+F 1 "PJ-3420" H 8970 4074 50  0000 R CNN
 F 2 "toripoyo:PJ-3420" H 9250 4050 50  0001 C CNN
 F 3 "~" H 9250 4050 50  0001 C CNN
@@
 	2100 5400 2100 5300
 Connection ~ 1800 5400
-Text GLabel 8550 3950 0    50   Input ~ 0
-BT_Line_out_L
-Text GLabel 8550 4050 0    50   Input ~ 0
-BT_Line_out_R
 $Comp
 L Device:R_Small R1
@@
 Wire Wire Line
 	9800 2050 9700 2050
+Text GLabel 8550 3950 0    50   Input ~ 0
+mix_out_L
+Text GLabel 8550 4050 0    50   Input ~ 0
+mix_out_R
 $EndSCHEMATC

Commit message: Rev.A 作成中
Parts:
- removed C3, C6, C9: 0.1u, Capacitor_SMD:C_0603_1608Metric_Pad1.05x0.95mm_HandSolder, symbol Device:C_Small
- renumbered R2 to R1, R12 to R10, R13 to R11, R14 to R12, R15 to R13, R16 to R14, R1 to R15, R5 to R16, R3 to R2, R4 to R3, R6 to R4, R7 to R5, R8 to R6, R9 to R7, R10 to R8, R11 to R9
Connections:
- net GND: now also RV1.1, RV1.4; no longer RV1.1, RV1.4
- net mix_out_L: now also RV1.3; no longer RV1.6
- net mix_out_R: now also RV1.6; no longer RV1.3
- net at U3.3 (+): now also RV1.2; no longer RV1.5
- net at U3.5 (+): now also RV1.5; no longer RV1.2
Other:
- moved on the sheet: C1, C2, C4, C5, C7, C8, U1C, U2C, U3C

Commit message: Rev.A 完成
Parts:
- removed H1, H2, H3, H4: MountingHole_Pad, MountingHole:MountingHole_3.2mm_M3_DIN965_Pad, symbol Mechanical:MountingHole_Pad
- added H1, H2, H3, H4: MountingHole, MountingHole:MountingHole_3.2mm_M3, symbol Mechanical:MountingHole
Changed lines of the file:
@@
 U 1 1 5EEA2F1E
 P 4600 2000
-F 0 "R7" V 4404 2000 50  0000 C CNN
-F 1 "47k" V 4500 2000 50  0000 C CNN
+F 0 "R7" V 4800 2000 50  0000 C CNN
+F 1 "47k" V 4700 2000 50  0000 C CNN
 F 2 "Resistor_SMD:R_0603_1608Metric_Pad1.05x0.95mm_HandSolder" H 4600 2000 50  0001 C CNN
 F 3 "~" H 4600 2000 50  0001 C CNN
@@
 $EndComp
 $Comp
-L Mechanical:MountingHole_Pad H1
-U 1 1 5F0C9455
-P 1200 5200
-F 0 "H1" H 1300 5249 50  0000 L CNN
-F 1 "MountingHole_Pad" H 1150 5600 50  0001 L CNN
-F 2 "MountingHole:MountingHole_3.2mm_M3_DIN965_Pad" H 1200 5200 50  0001 C CNN
-F 3 "~" H 1200 5200 50  0001 C CNN
-	1    1200 5200
-	1    0    0    -1
-$EndComp
-$Comp
-L Mechanical:MountingHole_Pad H2
-U 1 1 5F0CA32C
-P 1500 5200
-F 0 "H2" H 1600 5249 50  0000 L CNN
-F 1 "MountingHole_Pad" H 1150 5400 50  0000 L CNN
-F 2 "MountingHole:MountingHole_3.2mm_M3_DIN965_Pad" H 1500 5200 50  0001 C CNN
-F 3 "~" H 1500 5200 50  0001 C CNN
-	1    1500 5200
-	1    0    0    -1
-$EndComp
-$Comp
-L Mechanical:MountingHole_Pad H3
-U 1 1 5F0CA5BB
-P 1800 5200
-F 0 "H3" H 1900 5249 50  0000 L CNN
-F 1 "MountingHole_Pad" H 1900 5158 50  0001 L CNN
-F 2 "MountingHole:MountingHole_3.2mm_M3_DIN965_Pad" H 1800 5200 50  0001 C CNN
-F 3 "~" H 1800 5200 50  0001 C CNN
-	1    1800 5200
-	1    0    0    -1
-$EndComp
-$Comp
-L Mechanical:MountingHole_Pad H4
-U 1 1 5F0CA769
-P 2100 5200
-F 0 "H4" H 2200 5249 50  0000 L CNN
-F 1 "MountingHole_Pad" H 2200 5158 50  0001 L CNN
-F 2 "MountingHole:MountingHole_3.2mm_M3_DIN965_Pad" H 2100 5200 50  0001 C CNN
-F 3 "~" H 2100 5200 50  0001 C CNN
-	1    2100 5200
-	1    0    0    -1
-$EndComp
-$Comp
-L power:GND #PWR02
-U 1 1 5F0CA9AD
-P 1200 5500
-F 0 "#PWR02" H 1200 5250 50  0001 C CNN
-F 1 "GND" H 1205 5327 50  0000 C CNN
-F 2 "" H 1200 5500 50  0001 C CNN
-F 3 "" H 1200 5500 50  0001 C CNN
-	1    1200 5500
-	1    0    0    -1
-$EndComp
-Wire Wire Line
-	1200 5500 1200 5400
-Wire Wire Line
-	1200 5400 1500 5400
-Wire Wire Line
-	1500 5400 1500 5300
-Connection ~ 1200 5400
-Wire Wire Line
-	1200 5400 1200 5300
-Wire Wire Line
-	1500 5400 1800 5400
-Wire Wire Line
-	1800 5400 1800 5300
-Connection ~ 1500 5400
-Wire Wire Line
-	1800 5400 2100 5400
-Wire Wire Line
-	2100 5400 2100 5300
-Connection ~ 1800 5400
-$Comp
 L Device:R_Small R15
 U 1 1 5F289EA8
@@
 Wire Wire Line
 	4650 7000 4650 7050
+$Comp
+L Mechanical:MountingHole H1
+U 1 1 5FC2B0F1
+P 1175 5200
+F 0 "H1" H 1275 5200 50  0000 L CNN
+F 1 "MountingHole" H 1275 5155 50  0001 L CNN
+F 2 "MountingHole:MountingHole_3.2mm_M3" H 1175 5200 50  0001 C CNN
+F 3 "~" H 1175 5200 50  0001 C CNN
+	1    1175 5200
+	1    0    0    -1
+$EndComp
+$Comp
+L Mechanical:MountingHole H2
+U 1 1 5FC2BE98
+P 1475 5200
+F 0 "H2" H 1575 5200 50  0000 L CNN
+F 1 "MountingHole" H 1575 5155 50  0001 L CNN
+F 2 "MountingHole:MountingHole_3.2mm_M3" H 1475 5200 50  0001 C CNN
+F 3 "~" H 1475 5200 50  0001 C CNN
+	1    1475 5200
+	1    0    0    -1
+$EndComp
+$Comp
+L Mechanical:MountingHole H3
+U 1 1 5FC2C151
+P 1775 5200
+F 0 "H3" H 1875 5200 50  0000 L CNN
+F 1 "MountingHole" H 1875 5155 50  0001 L CNN
+F 2 "MountingHole:MountingHole_3.2mm_M3" H 1775 5200 50  0001 C CNN
+F 3 "~" H 1775 5200 50  0001 C CNN
+	1    1775 5200
+	1    0    0    -1
+$EndComp
+$Comp
+L Mechanical:MountingHole H4
+U 1 1 5FC2C38E
+P 2075 5200
+F 0 "H4" H 2175 5200 50  0000 L CNN
+F 1 "MountingHole" H 2175 5155 50  0001 L CNN
+F 2 "MountingHole:MountingHole_3.2mm_M3" H 2075 5200 50  0001 C CNN
+F 3 "~" H 2075 5200 50  0001 C CNN
+	1    2075 5200
+	1    0    0    -1
+$EndComp
 $EndSCHEMATC

Commit message: Rev.B 改版完了
Parts:
- added C19, C20: 22p, Capacitor_SMD:C_0603_1608Metric_Pad1.05x0.95mm_HandSolder, symbol Device:C_Small
Connections:
- net at R7.1, R9.2, U1.1: now also C19.1
- net at R1.1, R2.1, R3.1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: now also C19.2
- net at R10.2, R8.1, U2.1: now also C20.1
- net at R4.1, R5.1, R6.1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: now also C20.2
Changed lines of the file:
@@
 U 1 1 5EEA2F1E
 P 4600 2000
-F 0 "R7" V 4800 2000 50  0000 C CNN
-F 1 "47k" V 4700 2000 50  0000 C CNN
+F 0 "R7" V 4525 2000 50  0000 C CNN
+F 1 "47k" V 4450 2000 50  0000 C CNN
 F 2 "Resistor_SMD:R_0603_1608Metric_Pad1.05x0.95mm_HandSolder" H 4600 2000 50  0001 C CNN
 F 3 "~" H 4600 2000 50  0001 C CNN
@@
 	1    0    0    -1
 $EndComp
+$Comp
+L Device:C_Small C20
+U 1 1 5FD6092F
+P 4600 3500
+AR Path="/5FD6092F" Ref="C20"  Part="1"
+AR Path="/5EF8073C/5FD6092F" Ref="C?"  Part="1"
+F 0 "C20" V 4800 3450 50  0000 L CNN
+F 1 "22p" V 4700 3425 50  0000 L CNN
+F 2 "Capacitor_SMD:C_0603_1608Metric_Pad1.05x0.95mm_HandSolder" H 4600 3500 50  0001 C CNN
+F 3 "~" H 4600 3500 50  0001 C CNN
+	1    4600 3500
+	0    1    1    0
+$EndComp
+Wire Wire Line
+	4500 3500 4150 3500
+Connection ~ 4150 3500
+Wire Wire Line
+	4700 3500 5050 3500
+Wire Wire Line
+	5050 3500 5050 3800
+Connection ~ 5050 3800
+$Comp
+L Device:C_Small C19
+U 1 1 5FD6A6DC
+P 4600 1700
+AR Path="/5FD6A6DC" Ref="C19"  Part="1"
+AR Path="/5EF8073C/5FD6A6DC" Ref="C?"  Part="1"
+F 0 "C19" V 4800 1650 50  0000 L CNN
+F 1 "22p" V 4700 1625 50  0000 L CNN
+F 2 "Capacitor_SMD:C_0603_1608Metric_Pad1.05x0.95mm_HandSolder" H 4600 1700 50  0001 C CNN
+F 3 "~" H 4600 1700 50  0001 C CNN
+	1    4600 1700
+	0    1    1    0
+$EndComp
+Wire Wire Line
+	4500 1700 4150 1700
+Connection ~ 4150 1700
+Wire Wire Line
+	4700 1700 5050 1700
+Wire Wire Line
+	5050 1700 5050 2000
+Connection ~ 5050 2000
 $EndSCHEMATC
