File: Power.sch (KiCad schematic (older format))
At the start: 25 parts, among them J11 Barrel_Jack_Switch, J3 USB_B_Micro, SW1 SW_SPDT, U4 MCW03, U5 MCW03, U6 NJM7809, U7 NJM7909

Commit message: 改版中
Parts:
- removed C10, C11: 4.7u, Capacitor_THT:CP_Radial_D6.3mm_P2.50mm, symbol Device:CP
- removed C12, C13, C18, C19, C53, C54, C55, C56: 100u/16V, Capacitor_THT:CP_Radial_D5.0mm_P2.00mm, symbol Device:CP
- added C10, C11: 220u/6.3V, Capacitor_SMD:C_1210_3225Metric_Pad1.42x2.65mm_HandSolder, symbol Device:C_Small
- added C12, C13, C18, C19, C20, C21, C22, C23, C24, C35: 47u, Capacitor_SMD:C_1210_3225Metric_Pad1.42x2.65mm_HandSolder, symbol Device:C_Small
- added JP1, JP2: NoReg, Jumper:SolderJumper-2_P1.3mm_Open_TrianglePad1.0x1.5mm, symbol Jumper:SolderJumper_2_Open
- added TP1: +9V, TestPoint:TestPoint_Pad_D1.5mm, symbol Connector:TestPoint
- added TP2: -9V, TestPoint:TestPoint_Pad_D1.5mm, symbol Connector:TestPoint
- C14, C15, C16, C17: value 0.1u -> 47u; footprint Capacitor_SMD:C_0603_1608Metric_Pad1.05x0.95mm_HandSolder -> Capacitor_SMD:C_1210_3225Metric_Pad1.42x2.65mm_HandSolder
- SW1: value SW_SPDT -> 2MS1-T1-B2-M7-S-E
Connections:
- wire segments 97 -> 114
Other:
- note added: "3225"
- note added: "All 16V\n3225"
- note added: "Power"
- moved on the sheet: C52, D1, J11, J3, R17, R18, SW1, U4, U5, U6, U7

Commit message: Rev.A 作成中
Parts:
- removed C22, C23: 47u, Capacitor_SMD:C_1210_3225Metric_Pad1.42x2.65mm_HandSolder, symbol Device:C_Small
- removed TP1: +9V, TestPoint:TestPoint_Pad_D1.5mm, symbol Connector:TestPoint
- removed TP2: -9V, TestPoint:TestPoint_Pad_D1.5mm, symbol Connector:TestPoint
- renumbered C52 to C10, C10 to C11, C11 to C12, C12 to C13, C13 to C14, C14 to C15, C15 to C16, C16 to C17, C17 to C18, C18 to C19, C19 to C20, C20 to C21, C21 to C22, C24 to C25, C35 to C26, J11 to J3, J3 to J4
Connections:
- net GND: now also C21.2, C22.1, C25.2, C26.1
Other:
- moved on the sheet: C21, C22

Commit message: Rev.A 完成
Parts:
- removed C13, C14, C19, C20, C25, C26: 47u, Capacitor_SMD:C_1210_3225Metric_Pad1.42x2.65mm_HandSolder, symbol Device:C_Small
- removed J3: Barrel_Jack_Switch, hastech:MJ-179P, symbol Connector:Barrel_Jack_Switch
- removed JP1, JP2: NoReg, Jumper:SolderJumper-2_P1.3mm_Open_TrianglePad1.0x1.5mm, symbol Jumper:SolderJumper_2_Open
- added C31: 0.1u, Capacitor_SMD:C_0603_1608Metric_Pad1.05x0.95mm_HandSolder, symbol Device:C_Small
- added J3: Conn_02x02_Counter_Clockwise, Connector_PinHeader_2.54mm:PinHeader_2x02_P2.54mm_Vertical, symbol Connector_Generic:Conn_02x02_Counter_Clockwise
- added JP1: UserShort, Jumper:SolderJumper-2_P1.3mm_Open_RoundedPad1.0x1.5mm, symbol kamiya:UserShort
- added R54: 100, Resistor_SMD:R_0603_1608Metric_Pad1.05x0.95mm_HandSolder, symbol Device:R_Small
- R17: value 1k -> 4.7k
Connections:
- net +5VD: no longer R17.2
- net -9VA: now also D1.1 (K)
- net GND: now also R17.2, C31.2, J3.1 (Pin_1), J3.2 (Pin_2), JP1.1, R54.2; no longer C10.2, C11.2, C12.2, D1.1 (K), J4.5 (GND), U4.1 (-Vin), U5.1 (-Vin)
- new net GNDD: C10.2, C11.2, C12.2, C31.1, J3.3 (Pin_3), J3.4 (Pin_4), J4.5 (GND), JP1.2, R54.1, U4.1 (-Vin), U5.1 (-Vin)
- no-connect marks 5 -> 4
Other:
- note added: "GND_Short"
- moved on the sheet: C10, C11, C12, C15, C16, C17, C18, C21, C22, D1, J4, R17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

Commit message: Rev.B 改版完了
Parts:
- removed J3: Conn_02x02_Counter_Clockwise, Connector_PinHeader_2.54mm:PinHeader_2x02_P2.54mm_Vertical, symbol Connector_Generic:Conn_02x02_Counter_Clockwise
- removed JP1: UserShort, Jumper:SolderJumper-2_P1.3mm_Open_RoundedPad1.0x1.5mm, symbol kamiya:UserShort
- added SW7: SW_SPDT, Button_Switch_THT:SW_Slide_1P2T_CK_OS102011MS2Q, symbol Switch:SW_SPDT
- C31: value 0.1u -> 22u/25V; footprint Capacitor_SMD:C_0603_1608Metric_Pad1.05x0.95mm_HandSolder -> Capacitor_SMD:C_0805_2012Metric_Pad1.15x1.40mm_HandSolder
- R54: value 100 -> 1k
Connections:
- net GND: now also SW7.2 (B)
- net GNDD: now also SW7.1 (A)
- no-connect marks 4 -> 5
Other:
- note added: "GND_Short / Isolate"
- note removed: "GND_Short"
Changed lines of the file:
@@
 U 1 1 5F42523D
 P 5350 3175
-F 0 "C11" H 5150 3225 50  0000 L CNN
+F 0 "C11" H 5150 3250 50  0000 L CNN
 F 1 "220u/6.3V" H 4900 3075 50  0000 L CNN
 F 2 "Capacitor_SMD:C_1210_3225Metric_Pad1.42x2.65mm_HandSolder" H 5350 3175 50  0001 C CNN
@@
 U 1 1 5F429C0D
 P 5350 4475
-F 0 "C12" H 5150 4525 50  0000 L CNN
+F 0 "C12" H 5150 4550 50  0000 L CNN
 F 1 "220u/6.3V" H 4900 4375 50  0000 L CNN
 F 2 "Capacitor_SMD:C_1210_3225Metric_Pad1.42x2.65mm_HandSolder" H 5350 4475 50  0001 C CNN
@@
 U 1 1 600298AD
 P 2775 4900
-F 0 "C31" H 2875 4850 50  0000 L CNN
-F 1 "0.1u" H 2850 4975 50  0000 L CNN
-F 2 "Capacitor_SMD:C_0603_1608Metric_Pad1.05x0.95mm_HandSolder" H 2775 4900 50  0001 C CNN
+F 0 "C31" H 2950 4850 50  0000 L CNN
+F 1 "22u/25V" H 2875 4975 50  0000 L CNN
+F 2 "Capacitor_SMD:C_0805_2012Metric_Pad1.15x1.40mm_HandSolder" H 2775 4900 50  0001 C CNN
 F 3 "~" H 2775 4900 50  0001 C CNN
 	1    2775 4900
@@
 U 1 1 600C2693
 P 3000 4900
-F 0 "R54" H 2875 4950 50  0000 C CNN
-F 1 "100" H 2875 4850 50  0000 C CNN
+F 0 "R54" H 2850 4875 50  0000 C CNN
+F 1 "1k" H 2850 4975 50  0000 C CNN
 F 2 "Resistor_SMD:R_0603_1608Metric_Pad1.05x0.95mm_HandSolder" H 3000 4900 50  0001 C CNN
 F 3 "~" H 3000 4900 50  0001 C CNN
@@
 Wire Wire Line
 	3250 2500 3250 2700
-$Comp
-L Connector_Generic:Conn_02x02_Counter_Clockwise J3
-U 1 1 5FB4BAF9
-P 3725 4850
-F 0 "J3" V 3729 4930 50  0000 L CNN
-F 1 "Conn_02x02_Counter_Clockwise" V 4225 4675 50  0000 L CNN
-F 2 "Connector_PinHeader_2.54mm:PinHeader_2x02_P2.54mm_Vertical" H 3725 4850 50  0001 C CNN
-F 3 "~" H 3725 4850 50  0001 C CNN
-	1    3725 4850
-	0    1    1    0
-$EndComp
-Wire Wire Line
-	3625 4650 3625 4525
-Wire Wire Line
-	3625 4525 3275 4525
-Connection ~ 3000 4525
-Wire Wire Line
-	3625 4525 3725 4525
-Wire Wire Line
-	3725 4525 3725 4650
-Connection ~ 3625 4525
-Wire Wire Line
-	3625 5150 3625 5275
-Wire Wire Line
-	3625 5275 3275 5275
-Connection ~ 3000 5275
-Wire Wire Line
-	3725 5150 3725 5275
-Wire Wire Line
-	3725 5275 3625 5275
-Connection ~ 3625 5275
-Text Notes 3825 5150 0    50   ~ 0
-GND_Short
-$Comp
-L kamiya:UserShort JP1
-U 1 1 5FBCD4DA
-P 3275 4925
-F 0 "JP1" V 3250 5003 60  0000 L CNN
-F 1 "UserShort" H 3225 4825 60  0001 C CNN
-F 2 "Jumper:SolderJumper-2_P1.3mm_Open_RoundedPad1.0x1.5mm" H 3325 4925 60  0001 C CNN
-F 3 "" H 3325 4925 60  0000 C CNN
-	1    3275 4925
-	0    1    1    0
-$EndComp
-Wire Wire Line
-	3275 4725 3275 4525
-Connection ~ 3275 4525
-Wire Wire Line
-	3275 4525 3000 4525
-Wire Wire Line
-	3275 5075 3275 5275
-Connection ~ 3275 5275
-Wire Wire Line
-	3275 5275 3000 5275
+Text Notes 3650 5150 0    50   ~ 0
+GND_Short / Isolate
 $Comp
 L power:GND #PWR0101
@@
 Wire Wire Line
 	7950 3825 8175 3825
+$Comp
+L Switch:SW_SPDT SW7
+U 1 1 5FD32303
+P 3450 4900
+F 0 "SW7" V 3404 5048 50  0000 L CNN
+F 1 "SW_SPDT" V 3495 5048 50  0000 L CNN
+F 2 "Button_Switch_THT:SW_Slide_1P2T_CK_OS102011MS2Q" H 3450 4900 50  0001 C CNN
+F 3 "~" H 3450 4900 50  0001 C CNN
+	1    3450 4900
+	0    1    1    0
+$EndComp
+NoConn ~ 3350 5100
+Wire Wire Line
+	3000 5275 3550 5275
+Wire Wire Line
+	3550 5275 3550 5100
+Connection ~ 3000 5275
+Wire Wire Line
+	3450 4700 3450 4525
+Wire Wire Line
+	3450 4525 3000 4525
+Connection ~ 3000 4525
 $EndSCHEMATC
